File: CDJ-MainBoard/audio_outputs.kicad_sch (KiCad schematic)
At the start: 21 parts, among them J2 PJ-611E 6.35mm jack, J3 J_RCA_L (white), J4 J_RCA_R (red), J5 PJ-320D 3.5mm jack, U2 PCM5122PW

Commit message: Add the simulation sheets for the DAC and buck, add the MCPs multiplexers and the analog ADC multiplexer
Parts:
- added C60: 10uF, PCM_JLCPCB:C_0805, symbol PCM_JLCPCB-Capacitors:0805,10uF,(2)
Connections:
- net GND: now also C60.2
- net at C10.1, U2.26 (LDOO): now also C60.1
Other:
- moved on the sheet: C10
