File: CDJ-MainBoard/CDJ-MainBoard.kicad_sch (KiCad schematic)
At the start: 18 parts, among them J1 J_FAN_PWM, SW1 DSWB05LHGET, SW2 PWR_BUT_CM5, U1 Compute_Module_5_Functional

Commit message: Add the simulation sheets for the DAC and buck, add the MCPs multiplexers and the analog ADC multiplexer
Parts:
- removed BT1: CR2032-BS-6-1, JLC2KiCad_lib-footprints:BAT-TH_CR2032-BS-6-1, symbol CR2032-BS-6-1:CR2032-BS-6-1
- removed C1: 100nF, Capacitor_SMD:C_0402_1005Metric, symbol Device:C_Small
- removed D1: PSC-1608U52GC-G4, JLC2KiCad_lib-footprints:LED0603-RD_GREEN, symbol PSC-1608U52GC-G4:PSC-1608U52GC-G4
- removed D2: XL-1608UBC-04, JLC2KiCad_lib-footprints:LED0603-RD_BLUE, symbol XL-1608UBC-04:XL-1608UBC-04
- removed J1: J_FAN_PWM, Connector_JST:JST_PH_B4B-PH-K_1x04_P2.00mm_Vertical, symbol Connector_Generic:Conn_01x04
- removed R1: 10kΩ, JLC2KiCad_lib-footprints:R0402, symbol Device:R
- removed R10: 3.3kΩ, JLC2KiCad_lib-footprints:R0402, symbol Device:R
- removed R2, R3: 5.1kΩ, JLC2KiCad_lib-footprints:R0402, symbol Device:R
- removed R4, R6: 220Ω, JLC2KiCad_lib-footprints:R0402, symbol Device:R
- removed R5, R7, R9: 2.2kΩ, JLC2KiCad_lib-footprints:R0402, symbol Device:R
- removed R8: 100Ω, JLC2KiCad_lib-footprints:R0402, symbol Device:R
- removed SW1: DSWB05LHGET, JLC2KiCad_lib-footprints:SW-TH_DSWB05LHGET, symbol DSWB05LHGET:DSWB05LHGET
- removed SW2: PWR_BUT_CM5, PCM_JLCPCB:SW_TS-1088-AR02016, symbol Switch:SW_Push
- removed U1: Compute_Module_5_Functional, kicad-thirdparty-footprints:CM5, symbol rpi-cm-5:Compute_Module_5_Functional
Connections:
- no-connect marks 26 -> 0
Other:
- added sheet Compute Module (cm5.kicad_sch)
- added sheet Sim_Buck (sim_buck.kicad_sch)
- added sheet Sim_DAC (sim_dac.kicad_sch)
- note removed: "Add usb multiplexer for screen and second usb3 on CDJ"
- note removed: "Switch states: System SW_OFF SW_ON ---------------------------- Wifi enabled disabled BT enabled disabled EEPROM writable locked Boot eMMC USB"
