File: CDJ-MainBoard/CDJ-MainBoard.kicad_pcb (KiCad board)
At the start: 4 copper layers, 250 x 160 mm, 193 parts, among them J1 J_FAN_PWM, J10 USB_DJ_STICK (USB3_A), J11 USB_SCREEN (USB3_A), J12 HR911130A, J13 PI HDMI_0 (HDMI_D_1.4 micro), J14 PI HDMI_0 (HDMI_D_1.4 micro), J15 TYPE-C-31-M-12, J16 J_JOGWHEEL, J17 J_HOTCUES, J18 J_LEFT_CTRLS, J19 J_RIGHT_CTRLS, J2 PJ-611E 6.35mm jack, J20 J_TOP_LEFT, J21 J_TOP_RIGHT, J3 J_RCA_L (white), J4 J_RCA_R (red), J5 PJ-320D 3.5mm jack, J6 J_ISP_ATMEGA, J7 J_I2C, J8 AUX POWER USB_A, J9 TYPE-C_16PIN_2MD(073), SW1 DSWB05LHGET, SW2 PWR_BUT_CM5, SW3 SW_MAIN_POWER, SW4 RESET_BTN, U1 Compute_Module_5_Functional, U10 AP2112K-3.3 DIGITAL PSU LDO, U11 AP2112K-3.3 ANALOG AUDIO LDO, U12 CH224K, U13 SY8368AQQC, U14 ATmega32U4-A (Arduino MIDI co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, U16 74HC4067PW,118, U17 PCM5122PW, U18 MCP23017T-E/SS, U19 MCP23017T-E/SS, U2 PCM5122PW, U3 AP2553W6-7, U4 AP2553W6-7, U5 AP2553W6-7, U6 USBLC6-2SC6, U7 USBLC6-2SC6, U8 USBLC6-2SC6, U9 AP2553W6-7, X1 X322516MLB4SI

Commit message: Route SD card and misc
Parts:
- removed U17: PCM5122PW, Package_SO:TSSOP-28_4.4x9.7mm_P0.65mm
- added C65: 100nF, PCM_JLCPCB:C_0402, F.Cu at (242.9, 87.5)
- added C66: 100nF, PCM_JLCPCB:C_0402, F.Cu at (242.8, 79.9)
- added C75: 100nF, PCM_JLCPCB:C_0402, F.Cu at (243.0, 73.1)
- added C76: 10uF, PCM_JLCPCB:C_0805, F.Cu at (254.4, 91.0)
- added Q1: AO3400A NFET, PCM_JLCPCB:Q_SOT-23, F.Cu at (248.9, 94.1)
- added Q2: SI2301CDS-T1-GE3 P-FET, PCM_JLCPCB:Q_SOT-23, F.Cu at (253.6, 94.1)
- added R69: 33Ω, PCM_JLCPCB:R_0402, F.Cu at (246.2, 84.4)
- added R70: 10kΩ, PCM_JLCPCB:R_0402, F.Cu at (246.2, 82.1)
- added R71: 10kΩ, PCM_JLCPCB:R_0402, F.Cu at (253.7, 98.8)
- added R72: 10kΩ, PCM_JLCPCB:R_0402, F.Cu at (246.2, 80.0)
- added R73: 10kΩ, PCM_JLCPCB:R_0402, F.Cu at (253.7, 97.6)
- added R74: 10kΩ, PCM_JLCPCB:R_0402, F.Cu at (249.0, 77.8)
- added R75: 10kΩ, PCM_JLCPCB:R_0402, F.Cu at (247.6, 87.6)
- added R76: 10kΩ, PCM_JLCPCB:R_0402, F.Cu at (247.6, 85.4)
- added U20: TF-15×15, JLC2KiCad_lib-footprints:TF-SMD_TF-15-15, F.Cu at (254.6, 81.8)
- added U21: USBLC6-2SC6-ES, JLC2KiCad_lib-footprints:SOT-23-6_L2.9-W1.6-P0.95-LS2.8-BR, F.Cu at (242.8, 75.7)
- added U22: USBLC6-2SC6-ES, JLC2KiCad_lib-footprints:SOT-23-6_L2.9-W1.6-P0.95-LS2.8-BR, F.Cu at (153.2, 17.0)
- added U23: USBLC6-2SC6-ES, JLC2KiCad_lib-footprints:SOT-23-6_L2.9-W1.6-P0.95-LS2.8-BR, F.Cu at (242.6, 82.9)
- U6, U7, U8: value USBLC6-2SC6 -> USBLC6-2SC6-ES; footprint PCM_JLCPCB:SOT-23-6_L2.9-W1.6-P0.95-LS2.8-BR -> JLC2KiCad_lib-footprints:SOT-23-6_L2.9-W1.6-P0.95-LS2.8-BR
- moved TP6 110.0 mm to (42.9, 79.6)
- moved BT1 101.6 mm to (175.8, 53.2), turned to 180 degrees
- moved U7 91.6 mm to (242.6, 90.1), turned to 180 degrees
- moved TP9 88.9 mm to (22.4, 61.8)
- moved TP8 87.0 mm to (18.8, 61.6)
- moved D2 81.5 mm to (219.1, 81.4)
- moved D1 80.3 mm to (205.3, 84.4)
- moved J1 80.3 mm to (199.2, 72.0)
- moved R3 80.3 mm to (208.3, 64.0)
- moved R4 80.3 mm to (195.3, 64.0)
- moved R5 80.3 mm to (212.1, 76.0)
- moved R6 80.3 mm to (212.3, 69.0)
- moved R8 80.3 mm to (203.8, 62.5)
- moved R9 80.3 mm to (199.8, 63.0)
- moved SW1 80.1 mm to (91.6, 55.2), turned to -90 degrees
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Connections:
- U1 pad 57: (no net) -> Net-(U1I-SD_CLK)
- U1 pad 61: (no net) -> /Compute Module/SD_DAT3
- U1 pad 62: (no net) -> /Compute Module/SD_CMD
- U1 pad 63: (no net) -> /Compute Module/SD_DAT0
- U1 pad 64: (no net) -> unconnected-(U1I-SD_DAT5-Pad64)
- U1 pad 67: (no net) -> /Compute Module/SD_DAT1
- U1 pad 68: (no net) -> unconnected-(U1I-SD_DAT4-Pad68)
- U1 pad 69: (no net) -> /Compute Module/SD_DAT2
- U1 pad 70: (no net) -> unconnected-(U1I-SD_DAT7-Pad70)
- U1 pad 72: (no net) -> unconnected-(U1I-SD_DAT6-Pad72)
- U1 pad 73: (no net) -> unconnected-(U1I-SD_VDD_Override-Pad73)
- U1 pad 75: (no net) -> /Compute Module/SD_PWR_ON
- U6 pad 1: Net-(J9-DN1) -> Net-(J11-D-)
- U6 pad 3: Net-(J9-DP1) -> Net-(J11-D+)
- U6 pad 4: /USB DJ Ports/USB_C_DJ_DP -> /USB DJ Ports/USB_SCR_DP
- U6 pad 6: /USB DJ Ports/USB_C_DJ_DM -> /USB DJ Ports/USB_SCR_DM
- U7 pad 1: Net-(J10-D-) -> /Compute Module/SD_DAT0
- U7 pad 3: Net-(J10-D+) -> /Compute Module/SD_DAT1
- U7 pad 4: /USB DJ Ports/USB_DJ_DP -> /Compute Module/SD_DAT1
- U7 pad 5: +5V -> +3.3V
- U7 pad 6: /USB DJ Ports/USB_DJ_DM -> /Compute Module/SD_DAT0
- U8 pad 1: Net-(J11-D-) -> Net-(J10-D-)
- U8 pad 3: Net-(J11-D+) -> Net-(J10-D+)
- U8 pad 4: /USB DJ Ports/USB_SCR_DP -> /USB DJ Ports/USB_DJ_DP
- U8 pad 6: /USB DJ Ports/USB_SCR_DM -> /USB DJ Ports/USB_DJ_DM
Routing:
- net +3.3V: track 13.1 -> 306.9 mm, vias 4 -> 11
- net /Compute Module/S_BT_GND: track 0.00 -> 53.0 mm, vias 0 -> 3
- net /Compute Module/S_BOOT_GND: track 0.00 -> 52.9 mm, vias 0 -> 3
- net /Compute Module/S_WIFI_GND: track 0.00 -> 50.7 mm, vias 0 -> 3
- net /Compute Module/S_EEPROM_WP_GND: track 0.00 -> 35.6 mm, vias 0 -> 2
- net Net-(U1J-VBAT): track 0.00 -> 33.6 mm
- net GND: track 146.0 -> 179.5 mm, vias 62 -> 73
- net /Compute Module/SD_VDD: track 0.00 -> 13.0 mm
- net /Compute Module/SD_DAT2: track 0.00 -> 8.03 mm
- net /Compute Module/SD_DAT3: track 0.00 -> 8.03 mm
- net /Compute Module/SD_PWR_ON: track 0.00 -> 7.99 mm, vias 0 -> 2
- net /Compute Module/SD_DAT1: track 0.00 -> 7.91 mm
- net /Compute Module/SD_DAT0: track 0.00 -> 6.78 mm
- net Net-(Q1-D): track 0.00 -> 6.45 mm
- net /Compute Module/SD_CMD: track 0.00 -> 5.54 mm
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Other:
- board size 250 x 160 mm -> 250.1 x 104 mm
