File: CDJ-MainBoard/sim_buck.kicad_sch (KiCad schematic)
At the start: 20 parts, among them U15 SY8368AQQC

Commit message: Route SD card and misc
Parts:
- U15: footprint footprint:QFN-12_L3.0-W3.0-P0.45-TL-EP -> (none)
Changed lines of the file:
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@@
 			)
 		)
-		(property "Footprint" "footprint:QFN-12_L3.0-W3.0-P0.45-TL-EP"
+		(property "Footprint" ""
 			(at 162.56 52.07 0)
 			(effects
