File: TriMiXxX_Arduino_MIDI_HID/midi-laser-pcb/midi-laser-pcb.kicad_sch (KiCad schematic)
At the start: 32 parts, among them J1 Jogwheel, J2 UART_PI, J3 PLAY_CUE, J4 TRACK_ENCODER, J5 LOOP_SIZE, J6 LOOP, J7 TEMPO, J8 I2C, SW1 Arduino_RST, U1 ProMicro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

Commit message: Update schematics for jlcpcb productions, new dims, and sunlu petgcf calibration
Parts:
- removed FID1, FID2, FID3, FID4, FID5, FID6: Fiducial, Fiducial:Fiducial_Cross_1.5mm_Mask2mm, symbol Mechanical:Fiducial
Connections:
- no-connect marks 20 -> 14

Commit message: Add some stuff
Connections:
- net RELOOP_BTN: now also U2.27 (GPA6)
- net UART_RX_FROM_PI: now also U1.2 (RX1/PD2); no longer R3.1, R4.1
- net UART_TX_TO_PI: now also R3.1, R4.1; no longer U1.1 (TX0/PD3)
- net at R3.2: now also U1.1 (TX0/PD3); no longer U1.2 (RX1/PD2)
- no-connect marks 14 -> 13
Other:
- moved on the sheet: R3, R4
Changed lines of the file:
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@@
 	)
 	(junction
-		(at 38.1 69.85)
-		(diameter 0)
-		(color 0 0 0 0)
-	)
-	(junction
 		(at 133.35 93.98)
 		(diameter 0)
@@
 		(color 0 0 0 0)
 	)
+	(junction
+		(at 66.04 59.69)
+		(diameter 0)
+		(color 0 0 0 0)
+	)
 	(no_connect
 		(at 118.11 86.36)
@@
 	)
 	(no_connect
-		(at 247.65 66.04)
-	)
-	(no_connect
 		(at 247.65 88.9)
 	)
@@
 	(wire
 		(pts
-			(xy 77.47 69.85) (xy 77.47 78.74)
+			(xy 82.55 59.69) (xy 82.55 76.2)
 		)
 		(stroke
@@
 	(wire
 		(pts
-			(xy 77.47 78.74) (xy 82.55 78.74)
-		)
-		(stroke
-			(width 0)
-			(type default)
-		)
-	)
-	(wire
-		(pts
 			(xy 118.11 81.28) (xy 130.81 81.28)
 		)
@@
 	(wire
 		(pts
-			(xy 38.1 69.85) (xy 67.31 69.85)
-		)
-		(stroke
-			(width 0)
-			(type default)
-		)
-	)
-	(wire
-		(pts
 			(xy 210.82 73.66) (xy 212.09 73.66)
 		)
@@
 	(wire
 		(pts
-			(xy 33.02 69.85) (xy 38.1 69.85)
+			(xy 60.96 59.69) (xy 66.04 59.69)
 		)
 		(stroke
@@
 	(wire
 		(pts
-			(xy 82.55 60.96) (xy 82.55 76.2)
+			(xy 130.81 77.47) (xy 135.89 77.47)
 		)
 		(stroke
@@
 	(wire
 		(pts
-			(xy 130.81 77.47) (xy 135.89 77.47)
+			(xy 66.04 59.69) (xy 72.39 59.69)
 		)
 		(stroke
@@
 	(wire
 		(pts
-			(xy 74.93 69.85) (xy 77.47 69.85)
+			(xy 80.01 59.69) (xy 82.55 59.69)
 		)
 		(stroke
@@
 		)
 	)
-	(label "UART_TX_TO_PI"
-		(at 82.55 60.96 180)
-		(effects
-			(font
-				(size 1.27 1.27)
-			)
-			(justify right bottom)
-		)
-	)
 	(label "LOOP_DBL_BTN"
 		(at 318.77 62.23 180)
@@
 		)
 	)
+	(label "UART_RX_FROM_PI"
+		(at 82.55 78.74 180)
+		(effects
+			(font
+				(size 1.27 1.27)
+			)
+			(justify right bottom)
+		)
+	)
 	(label "LED_PLAY"
 		(at 247.65 78.74 0)
@@
 		)
 	)
+	(label "UART_TX_TO_PI"
+		(at 60.96 59.69 180)
+		(effects
+			(font
+				(size 1.27 1.27)
+			)
+			(justify right bottom)
+		)
+	)
 	(label "LOOP_HLF_BTN"
 		(at 318.77 59.69 180)
@@
 		)
 	)
-	(label "UART_RX_FROM_PI"
-		(at 33.02 69.85 180)
+	(label "JOG2"
+		(at 379.73 93.98 180)
 		(effects
 			(font
@@
 		)
 	)
-	(label "JOG2"
-		(at 379.73 93.98 180)
+	(label "ENC_SW"
+		(at 321.31 33.02 180)
 		(effects
 			(font
@@
 		)
 	)
-	(label "ENC_SW"
-		(at 321.31 33.02 180)
+	(label "RELOOP_BTN"
+		(at 247.65 66.04 0)
 		(effects
 			(font
 				(size 1.27 1.27)
 			)
-			(justify right bottom)
+			(justify left bottom)
 		)
 	)
@@
 	(symbol
 		(lib_id "Device:R")
-		(at 71.12 69.85 90)
+		(at 76.2 59.69 90)
 		(unit 1)
 		(body_style 1)
@@
 		(in_pos_files yes)
 		(dnp no)
-		(fields_autoplaced yes)
 		(property "Reference" "R3"
-			(at 71.12 63.5 90)
+			(at 76.2 53.34 90)
 			(show_name no)
 			(do_not_autoplace no)
@@
 		)
 		(property "Value" "4.7k"
-			(at 71.12 66.04 90)
+			(at 76.2 55.88 90)
 			(show_name no)
 			(do_not_autoplace no)
@@
 		)
 		(property "Footprint" "Resistor_THT:R_Axial_DIN0207_L6.3mm_D2.5mm_P10.16mm_Horizontal"
-			(at 71.12 71.628 90)
+			(at 76.2 61.468 90)
 			(hide yes)
 			(show_name no)
@@
 		)
 		(property "Datasheet" ""
-			(at 71.12 69.85 0)
+			(at 76.2 59.69 0)
 			(hide yes)
 			(show_name no)
@@
 		)
 		(property "Description" "Resistor"
-			(at 71.12 69.85 0)
+			(at 76.2 59.69 0)
 			(hide yes)
 			(show_name no)
@@
 	(symbol
 		(lib_id "power:GND")
-		(at 38.1 77.47 0)
+		(at 66.04 67.31 0)
 		(unit 1)
 		(body_style 1)
@@
 		(fields_autoplaced yes)
 		(property "Reference" "#PWR023"
-			(at 38.1 83.82 0)
+			(at 66.04 73.66 0)
 			(hide yes)
 			(show_name no)
@@
 		)
 		(property "Value" "GND"
-			(at 38.1 82.55 0)
+			(at 66.04 72.39 0)
 			(show_name no)
 			(do_not_autoplace no)
@@
 		)
 		(property "Footprint" ""
-			(at 38.1 77.47 0)
+			(at 66.04 67.31 0)
 			(hide yes)
 			(show_name no)
@@
 		)
 		(property "Datasheet" ""
-			(at 38.1 77.47 0)
+			(at 66.04 67.31 0)
 			(hide yes)
 			(show_name no)
@@
 		)
 		(property "Description" "Power symbol creates a global label with name \"GND\" , ground"
-			(at 38.1 77.47 0)
+			(at 66.04 67.31 0)
 			(hide yes)
 			(show_name no)
@@
 	(symbol
 		(lib_id "Device:R")
-		(at 38.1 73.66 0)
+		(at 66.04 63.5 0)
 		(unit 1)
 		(body_style 1)
@@
 		(fields_autoplaced yes)
 		(property "Reference" "R4"
-			(at 40.64 72.3899 0)
+			(at 68.58 62.2299 0)
 			(show_name no)
 			(do_not_autoplace no)
@@
 		)
 		(property "Value" "10k"
-			(at 40.64 74.9299 0)
+			(at 68.58 64.7699 0)
 			(show_name no)
 			(do_not_autoplace no)
@@
 		)
 		(property "Footprint" "Resistor_THT:R_Axial_DIN0207_L6.3mm_D2.5mm_P10.16mm_Horizontal"
-			(at 36.322 73.66 90)
+			(at 64.262 63.5 90)
 			(hide yes)
 			(show_name no)
@@
 		)
 		(property "Datasheet" ""
-			(at 38.1 73.66 0)
+			(at 66.04 63.5 0)
 			(hide yes)
 			(show_name no)
@@
 		)
 		(property "Description" "Resistor"
-			(at 38.1 73.66 0)
+			(at 66.04 63.5 0)
 			(hide yes)
 			(show_name no)
