File: TriMiXxX_Arduino_MIDI_HID/one_button/OneButton.kicad_pcb (KiCad board)
At the start: 2 copper layers, 20 x 20 mm, 18 parts, among them J1 INPUT, J2 OUTPUT, SW1 TS-1187A-B-A-B, U1 CH32V003F4U6

Commit message: Init trimixxx-midi platformIO project
Parts:
- turned R1 to 0 degrees
Connections:
- R1 pad 1: Net-(U1-PC0) -> /LED1_DIN
- R1 pad 2: /LED1_DIN -> Net-(U1-PC6)
- U1 pad 13: unconnected-(U1-PC6-Pad13) -> Net-(U1-PC6)
- U1 pad 7: Net-(U1-PC0) -> unconnected-(U1-PC0-Pad7)
Routing:
- net Net-(U1-PC6): track 0.00 -> 15.5 mm, vias 0 -> 2
- net Net-(U1-PC0): track 12.3 -> 0.00 mm, vias 2 -> 0
- net /SWIO: track 24.8 -> 25.7 mm
Other:
- board text added: "OneButton Rev V2.0 2026-07-07"
- board text removed: "OneButton Rev V1.0 2026-06-29"
