File: TriMiXxX_Arduino_MIDI_HID/midi_s3_mini/midi_s3_mini/jogb_assy.kicad_sch (KiCad schematic)
At the start: 7 parts, among them J13 Conn_01x04, J14 GP1A038RBK

Commit message: I'm not sure
Parts:
- R6: value R2202 -> R2202 100 ohms
- R7: value R2201 -> R2201 100 ohms
- R8: value R2203 -> R2203 330ohms
Changed lines of the file:
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@@
 			)
 		)
-		(property "Value" "R2203"
+		(property "Value" "R2203 330ohms"
 			(at 71.12 87.63 90)
 			(show_name no)
@@
 			)
 		)
-		(property "Value" "R2202"
+		(property "Value" "R2202 100 ohms"
 			(at 124.46 45.72 90)
 			(show_name no)
@@
 			)
 		)
-		(property "Value" "R2201"
+		(property "Value" "R2201 100 ohms"
 			(at 124.46 55.88 90)
 			(show_name no)
