File: TriMiXxX_Arduino_MIDI_HID/midi_s3_mini/midi_s3_mini/midi_s3_mini.kicad_sch (KiCad schematic)
At the start: 31 parts, among them J1 Power, J10 OneButtonA_TX, J11 OneButtonB_RX, J2 LOOP, J3 PLAY_CUE, J4 UART_PI, J5 TRACK_ENC, J6 TEMPO, J7 JOG, J8 OneButtonB_TX, J9 OneButtonA_RX, U1 LOLIN_S3_Mini

Commit message: Add Midi S3 Mini board V3
Parts:
- added C13, C8: 100n, easyeda2kicad:CAP-TH_L4.2-W3.5-P2.54-D0.5, symbol easyeda2kicad:178MU0006
- added J1: Power2, easyeda2kicad:CONN-TH_S2B-PH-K-S-LF-SN, symbol easyeda2kicad:S2B-PH-K-S
- added R5: 10k, easyeda2kicad:RES-TH_BD2.5-L6.5-P10.50-D0.6, symbol easyeda2kicad:MFR0W4F1002A50
- J2: renamed from J1; value Power -> Power1
- renumbered C7 to C12, C4 to C3, C8 to C4, C3 to C5, C5 to C7, H2 to H1, H1 to H2, J3 to J10, J7 to J11, J6 to J12, J4 to J3, J10 to J4, J9 to J5, J11 to J6, J8 to J7, J2 to J8, J5 to J9, R3 to R1, R1 to R2, R4 to R3, R2 to R4
Connections:
- net +3.3V: now also C11.2, J11.3, J12.1, C13.2, R5.2; no longer J11.2, J12.2
- net +5V: now also J1.1; no longer C11.2
- net BTN_CUE: now also U1.28 (IO35/SDA); no longer U1.21 (IO21)
- net BTN_PLAY: now also U1.21 (IO21); no longer U1.27 (IO36/SCL)
- net ENC_CLK: now also J9.5; no longer J9.3
- net ENC_SW: now also J9.3; no longer J9.5
- net GND: now also J11.2, J12.4, C13.1, C8.1, J1.2; no longer J11.1, J12.1
- net JOG1: now also J11.5; no longer J11.3
- net JOG_TCH: now also J11.1, C8.2, R5.1; no longer J11.5
- net LED_CUE: now also U1.27 (IO36/SCL); no longer U1.29 (IO18)
- net LED_PLAY: now also U1.29 (IO18); no longer U1.28 (IO35/SDA)
- net TEMPO_ADCT: now also J12.2, U1.14 (IO8); no longer J12.4, U1.15 (IO9)
- net TEMPO_ADIN: now also U1.15 (IO9); no longer U1.14 (IO8)
Other:
- note added: "Optical enc is used to be +5V, just should run fine at +3.3V TCH is normally opened, and GND when closed. Closed it has a 33ohms R to GND"
- note added: "Originally meant for 5V, but fully passive potentiometer, so works at 3.3V"
- note added: "This pinout matches the encoder's pinout if I mount a JST-PH angled on its bottom side"
- note removed: "TODO: Is the optical enc able to take in/output 3.3V, or only 5V?"
- note removed: "TODO: check the pinout order of the tempo board"
- moved on the sheet: C7, H1, H2, H3, H4, J11, J12, J3, J4, J5, J6, J7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

Commit message: Add Jogwheel lib and schematic for jogb assy
Other:
- added sheet JOGB_ASSY (jogb_assy.kicad_sch)
Changed lines of the file:
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@@
+		)
+	)
+	(sheet
+		(at 243.84 133.35)
+		(size 38.1 26.67)
+		(exclude_from_sim yes)
+		(in_bom no)
+		(on_board no)
+		(dnp yes)
+		(fields_autoplaced yes)
+		(stroke
+			(width 0.1524)
+			(type solid)
+		)
+		(fill
+			(color 0 0 0 0)
+		)
+		(property "Sheetname" "JOGB_ASSY"
+			(at 243.84 132.6384 0)
+			(show_name no)
+			(do_not_autoplace no)
+			(effects
+				(font
+					(size 1.27 1.27)
+				)
+				(justify left bottom)
+			)
+		)
+		(property "Sheetfile" "jogb_assy.kicad_sch"
+			(at 243.84 160.6046 0)
+			(show_name no)
+			(do_not_autoplace no)
+			(effects
+				(font
+					(size 1.27 1.27)
+				)
+				(justify left top)
+			)
+		)
+		(instances
+			(project "midi_s3_mini"
+				(path "/4a4c0c1b-df1c-48df-9685-1cfae0dce3a5"
+					(page "2")
+				)
+			)
 		)
 	)
