File: boards/midi_s3_mini/jogb_assy.kicad_sch (KiCad schematic)
At the start: 7 parts, among them J13 Conn_01x04, J14 GP1A038RBK

Commit message: Finish the ESD and power system for the V2 midi S3
Parts:
- renumbered C14 to C12, C15 to C13, J14 to J11, J13 to J12, R6 to R27, R7 to R28, R8 to R29
Changed lines of the file:
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@@
 		(in_pos_files yes)
 		(dnp no)
-		(property "Reference" "#PWR057"
+		(property "Reference" "#PWR059"
 			(at 105.41 83.82 0)
 			(hide yes)
@@
 			(project "midi_s3_mini"
 				(path "/4a4c0c1b-df1c-48df-9685-1cfae0dce3a5/000082a9-0d26-4c90-bc70-4bba8221bfab"
-					(reference "#PWR057")
+					(reference "#PWR059")
 					(unit 1)
 				)
@@
 		(dnp no)
 		(fields_autoplaced yes)
-		(property "Reference" "R8"
+		(property "Reference" "R29"
 			(at 71.12 85.09 90)
 			(show_name no)
@@
 			(project "midi_s3_mini"
 				(path "/4a4c0c1b-df1c-48df-9685-1cfae0dce3a5/000082a9-0d26-4c90-bc70-4bba8221bfab"
-					(reference "R8")
+					(reference "R29")
 					(unit 1)
 				)
@@
 		(dnp no)
 		(fields_autoplaced yes)
-		(property "Reference" "C14"
+		(property "Reference" "C12"
 			(at 109.22 82.5499 0)
 			(show_name no)
@@
 			(project "midi_s3_mini"
 				(path "/4a4c0c1b-df1c-48df-9685-1cfae0dce3a5/000082a9-0d26-4c90-bc70-4bba8221bfab"
-					(reference "C14")
+					(reference "C12")
 					(unit 1)
 				)
@@
 		(dnp no)
 		(fields_autoplaced yes)
-		(property "Reference" "R6"
+		(property "Reference" "R27"
 			(at 124.46 43.18 90)
 			(show_name no)
@@
 			(project "midi_s3_mini"
 				(path "/4a4c0c1b-df1c-48df-9685-1cfae0dce3a5/000082a9-0d26-4c90-bc70-4bba8221bfab"
-					(reference "R6")
+					(reference "R27")
 					(unit 1)
 				)
@@
 		(dnp no)
 		(fields_autoplaced yes)
-		(property "Reference" "#PWR058"
+		(property "Reference" "#PWR063"
 			(at 76.2 105.41 0)
 			(hide yes)
@@
 			(project "midi_s3_mini"
 				(path "/4a4c0c1b-df1c-48df-9685-1cfae0dce3a5/000082a9-0d26-4c90-bc70-4bba8221bfab"
-					(reference "#PWR058")
+					(reference "#PWR063")
 					(unit 1)
 				)
@@
 		(dnp no)
 		(fields_autoplaced yes)
-		(property "Reference" "#PWR055"
+		(property "Reference" "#PWR061"
 			(at 125.73 88.9 0)
 			(hide yes)
@@
 			(project "midi_s3_mini"
 				(path "/4a4c0c1b-df1c-48df-9685-1cfae0dce3a5/000082a9-0d26-4c90-bc70-4bba8221bfab"
-					(reference "#PWR055")
+					(reference "#PWR061")
 					(unit 1)
 				)
@@
 		(dnp no)
 		(fields_autoplaced yes)
-		(property "Reference" "#PWR054"
+		(property "Reference" "#PWR060"
 			(at 129.54 80.01 0)
 			(hide yes)
@@
 			(project "midi_s3_mini"
 				(path "/4a4c0c1b-df1c-48df-9685-1cfae0dce3a5/000082a9-0d26-4c90-bc70-4bba8221bfab"
-					(reference "#PWR054")
+					(reference "#PWR060")
 					(unit 1)
 				)
@@
 		(dnp no)
 		(fields_autoplaced yes)
-		(property "Reference" "#PWR056"
+		(property "Reference" "#PWR062"
 			(at 105.41 93.98 0)
 			(hide yes)
@@
 			(project "midi_s3_mini"
 				(path "/4a4c0c1b-df1c-48df-9685-1cfae0dce3a5/000082a9-0d26-4c90-bc70-4bba8221bfab"
-					(reference "#PWR056")
+					(reference "#PWR062")
 					(unit 1)
 				)
@@
 		(dnp no)
 		(fields_autoplaced yes)
-		(property "Reference" "J13"
+		(property "Reference" "J12"
 			(at 133.35 77.4699 0)
 			(show_name no)
@@
 			(project "midi_s3_mini"
 				(path "/4a4c0c1b-df1c-48df-9685-1cfae0dce3a5/000082a9-0d26-4c90-bc70-4bba8221bfab"
-					(reference "J13")
+					(reference "J12")
 					(unit 1)
 				)
@@
 		(dnp no)
 		(fields_autoplaced yes)
-		(property "Reference" "C15"
+		(property "Reference" "C13"
 			(at 80.01 93.9799 0)
 			(show_name no)
@@
 			(project "midi_s3_mini"
 				(path "/4a4c0c1b-df1c-48df-9685-1cfae0dce3a5/000082a9-0d26-4c90-bc70-4bba8221bfab"
-					(reference "C15")
+					(reference "C13")
 					(unit 1)
 				)
@@
 		(dnp no)
 		(fields_autoplaced yes)
-		(property "Reference" "R7"
+		(property "Reference" "R28"
 			(at 124.46 53.34 90)
 			(show_name no)
@@
 			(project "midi_s3_mini"
 				(path "/4a4c0c1b-df1c-48df-9685-1cfae0dce3a5/000082a9-0d26-4c90-bc70-4bba8221bfab"
-					(reference "R7")
+					(reference "R28")
 					(unit 1)
 				)
@@
 		(dnp no)
 		(fields_autoplaced yes)
-		(property "Reference" "J14"
+		(property "Reference" "J11"
 			(at 76.2 35.56 0)
 			(show_name no)
@@
 			(project "midi_s3_mini"
 				(path "/4a4c0c1b-df1c-48df-9685-1cfae0dce3a5/000082a9-0d26-4c90-bc70-4bba8221bfab"
-					(reference "J14")
+					(reference "J11")
 					(unit 1)
 				)
@@
 		(dnp no)
 		(fields_autoplaced yes)
-		(property "Reference" "#PWR059"
+		(property "Reference" "#PWR058"
 			(at 82.55 71.12 0)
 			(hide yes)
@@
 			(project "midi_s3_mini"
 				(path "/4a4c0c1b-df1c-48df-9685-1cfae0dce3a5/000082a9-0d26-4c90-bc70-4bba8221bfab"
-					(reference "#PWR059")
-					(unit 1)
-				)
+					(reference "#PWR058")
+					(unit 1)
+				)

Commit message: Footprint assignment for SMD assy
Parts:
- renumbered C12 to C11, C13 to C12
Changed lines of the file:
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@@
 		(in_pos_files yes)
 		(dnp no)
-		(property "Reference" "#PWR059"
+		(property "Reference" "#PWR057"
 			(at 105.41 83.82 0)
 			(hide yes)
@@
 			(project "midi_s3_mini"
 				(path "/4a4c0c1b-df1c-48df-9685-1cfae0dce3a5/000082a9-0d26-4c90-bc70-4bba8221bfab"
-					(reference "#PWR059")
+					(reference "#PWR057")
 					(unit 1)
 				)
@@
 		(dnp no)
 		(fields_autoplaced yes)
-		(property "Reference" "C12"
+		(property "Reference" "C11"
 			(at 109.22 82.5499 0)
 			(show_name no)
@@
 			(project "midi_s3_mini"
 				(path "/4a4c0c1b-df1c-48df-9685-1cfae0dce3a5/000082a9-0d26-4c90-bc70-4bba8221bfab"
-					(reference "C12")
+					(reference "C11")
 					(unit 1)
 				)
@@
 		(dnp no)
 		(fields_autoplaced yes)
-		(property "Reference" "#PWR063"
+		(property "Reference" "#PWR061"
 			(at 76.2 105.41 0)
 			(hide yes)
@@
 			(project "midi_s3_mini"
 				(path "/4a4c0c1b-df1c-48df-9685-1cfae0dce3a5/000082a9-0d26-4c90-bc70-4bba8221bfab"
-					(reference "#PWR063")
+					(reference "#PWR061")
 					(unit 1)
 				)
@@
 		(dnp no)
 		(fields_autoplaced yes)
-		(property "Reference" "#PWR061"
+		(property "Reference" "#PWR059"
 			(at 125.73 88.9 0)
 			(hide yes)
@@
 			(project "midi_s3_mini"
 				(path "/4a4c0c1b-df1c-48df-9685-1cfae0dce3a5/000082a9-0d26-4c90-bc70-4bba8221bfab"
-					(reference "#PWR061")
+					(reference "#PWR059")
 					(unit 1)
 				)
@@
 		(dnp no)
 		(fields_autoplaced yes)
-		(property "Reference" "#PWR060"
+		(property "Reference" "#PWR058"
 			(at 129.54 80.01 0)
 			(hide yes)
@@
 			(project "midi_s3_mini"
 				(path "/4a4c0c1b-df1c-48df-9685-1cfae0dce3a5/000082a9-0d26-4c90-bc70-4bba8221bfab"
-					(reference "#PWR060")
+					(reference "#PWR058")
 					(unit 1)
 				)
@@
 		(dnp no)
 		(fields_autoplaced yes)
-		(property "Reference" "#PWR062"
+		(property "Reference" "#PWR060"
 			(at 105.41 93.98 0)
 			(hide yes)
@@
 			(project "midi_s3_mini"
 				(path "/4a4c0c1b-df1c-48df-9685-1cfae0dce3a5/000082a9-0d26-4c90-bc70-4bba8221bfab"
-					(reference "#PWR062")
+					(reference "#PWR060")
 					(unit 1)
 				)
@@
 		(dnp no)
 		(fields_autoplaced yes)
-		(property "Reference" "C13"
+		(property "Reference" "C12"
 			(at 80.01 93.9799 0)
 			(show_name no)
@@
 			(project "midi_s3_mini"
 				(path "/4a4c0c1b-df1c-48df-9685-1cfae0dce3a5/000082a9-0d26-4c90-bc70-4bba8221bfab"
-					(reference "C13")
+					(reference "C12")
 					(unit 1)
 				)
@@
 		(dnp no)
 		(fields_autoplaced yes)
-		(property "Reference" "#PWR058"
+		(property "Reference" "#PWR056"
 			(at 82.55 71.12 0)
 			(hide yes)
@@
 			(project "midi_s3_mini"
 				(path "/4a4c0c1b-df1c-48df-9685-1cfae0dce3a5/000082a9-0d26-4c90-bc70-4bba8221bfab"
-					(reference "#PWR058")
-					(unit 1)
-				)
+					(reference "#PWR056")
+					(unit 1)
+				)
