File: boards/midi_s3_mini/midi_s3_mini.kicad_pcb (KiCad board)
At the start: 2 copper layers, 90 x 70 mm, 102 parts, among them J1 1BTN_A_TX, J10 JOG, J13 PowerIn, J14 TEST_5V, J15 GND_IN, J16 TEST_3V3_S3, J17 TEST_3V3_PERI, J18 GND_PERI, J2 1BTN_A_RX, J3 1BN_B_RX, J4 1BTN_B_TX, J5 UART_PI, J6 TRACK_ENC, J7 LOOP, J8 PLAY_CUE, J9 TEMPO, Q1 AO3401A, U1 LOLIN_S3_Mini, U2 SPX3819M5-L/TR

Commit message: Add my custom graphics
Other:
- board text added: "TriMiXxX S3 MIDI Control Board V2"
- board text removed: "TriMiXxX MIDI Control Board V3"

Commit message: Finally fabbed v2
Parts:
- C_LDO_out1: value 2.2uF (225) ±20% 50V -> 2.2uF ±10% 50V
- J3: value 1BN_B_RX -> 1BTN_B_RX
- moved C_LDO_out1 0.10 mm to (83.5, 34.0)
- moved R33 0.07 mm to (84.7, 36.5)
- renumbered D_S1 to D3, D_PERI1 to D4
