File: boards/midi_s3_mini/power.kicad_sch (KiCad schematic)
At the start: 21 parts, among them J1 PowerIn, Q1 AO3401A, U2 SPX3819M5-L/TR

Commit message: Add test points and leds
Parts:
- added J15: TEST_3V3_S3, symbol Connector:Conn_01x01_Pin
- added J16: TEST_3V3_PERI, symbol Connector:Conn_01x01_Pin
- added J17: GND_IN, symbol Connector:Conn_01x01_Pin
- added J18: GND_PERI, symbol Connector:Conn_01x01_Pin
- added J2: TEST_5V, symbol Connector:Conn_01x01_Pin
- added LED_3V3_PERI: Yellow, easyeda2kicad:LED0805-R-RD, symbol easyeda2kicad:17-21SUYC_TR8
- added LED_3V3_S3: Green, easyeda2kicad:LED0805-R-RD, symbol easyeda2kicad:0805G
- added LED_5V: Red, easyeda2kicad:LED0805-RD, symbol easyeda2kicad:FC-2012HRK-620D
- added R12: 3.3KΩ ±1%, easyeda2kicad:R0402, symbol easyeda2kicad:0402WGF3301TCE
- added R14: 470Ω ±1%, easyeda2kicad:R0402, symbol easyeda2kicad:0402WGF4700TCE
- added R15: 1.5KΩ ±1%, easyeda2kicad:R0402, symbol easyeda2kicad:0402WGF1501TCE
- added TP1: VIN_5V, symbol Connector:TestPoint
- added TP2: LDO_OUT, symbol Connector:TestPoint
- renumbered D_periph to D_PERI
Connections:
- net +3.3V: now also J16.1 (Pin_1), R15.2
- net +5V: now also J2.1 (Pin_1), R12.2
- net GND: now also J17.1 (Pin_1), J18.1 (Pin_1), LED_3V3_PERI.2 (-), LED_3V3_S3.2 (K), LED_5V.1 (-)
- net LDO_OUT_3.6V: now also TP2.1
- net S3_3.3V: now also J15.1 (Pin_1), R14.2
- net VIN_5V: now also TP1.1
- new net: LED_3V3_S3.1 (A), R14.1
- new net: LED_5V.2 (+), R12.1
- new net: LED_3V3_PERI.1 (+), R15.1
Other:
- moved on the sheet: C16, C17, C3, C5, C_LDO_in, C_LDO_out, D2, D_PERI, JP1, R10, R11, R9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

Commit message: Finish the ESD and power system for the V2 midi S3
Parts:
- removed C3: 100n, easyeda2kicad:CAP-TH_L4.2-W3.5-P2.54-D0.5, symbol easyeda2kicad:178MU0006
- added C16, C20: 100n s, easyeda2kicad:C0402, symbol easyeda2kicad:CL05B104KB54PNC
- renumbered C6 to C14, C2 to C15, C5 to C17, C16 to C18, C17 to C19, C18 to C21, C_LDO_in to C_LDO_in1, C_LDO_out to C_LDO_out1, D_PERI to D_PERI1, D_S3 to D_S1, J1 to J13, J2 to J14, J17 to J15, J15 to J16, J16 to J17, LED_3V3_PERI to LED_3V3_PERI1, LED_3V3_S3 to LED_3V3_S1, LED_5V to LED_5V1, R12 to R30, R13 to R31, R9 to R32, R10 to R33, R11 to R34, R14 to R35, R15 to R36, TP1 to TP2, TP2 to TP3
Connections:
- net +5V: now also C16.2
- net GND: now also C16.1, C20.2
- net S3_3.3V: now also C20.1

Commit message: Footprint assignment for SMD assy
Parts:
- removed C14: 100n, easyeda2kicad:CAP-TH_L4.2-W3.5-P2.54-D0.5, symbol easyeda2kicad:178MU0006
- removed R32: 47k, symbol Device:R_Small
- removed R33: 24k, symbol Device:R_Small
- added C21: 100n, easyeda2kicad:C0402, symbol easyeda2kicad:CL05B104KB54PNC
- added R3: 22KΩ ±1%, easyeda2kicad:R0402, symbol easyeda2kicad:0402WGF2202TCE
- added R4: 47KΩ ±1%, easyeda2kicad:R0402, symbol easyeda2kicad:0402WGF4702TCE
- C15: renamed from C16; value 100n s -> 100n
- C19: renamed from C20; value 100n s -> 100n
- J13: footprint (none) -> TerminalBlock_Altech:Altech_AK300_1x02_P5.00mm_45-Degree
- J14, J15, J16, J17, J18: footprint (none) -> Connector_PinHeader_2.54mm:PinHeader_1x01_P2.54mm_Vertical
- JP1: footprint (none) -> Connector_PinHeader_2.54mm:PinHeader_1x02_P2.54mm_Vertical
- TP2, TP3: footprint (none) -> TestPoint:TestPoint_Pad_D2.5mm
- renumbered C15 to C14, C17 to C16, C18 to C17, C19 to C18, C21 to C20
Connections:
- net GND: now also C21.1, R3.1
- net VIN_5V: now also C21.2
- net at U2.4 (ADJ/BYP): now also R3.2, R4.1
- net LDO_OUT_3.6V renamed LDO_OUT
- net LDO_OUT: now also R4.2
Other:
- note added: "Main 3V3 LDO, provides up to 500mA (enough for WiFi) Be careful with ADC tempo noise! Set to LDO output strictly more than 3.3V The schotky drops 550mV which wins over the 3.3V of the USB. When externally powered + USB powered, this means the USB power loses and the ext takes over. ~300 µVrms in adjustable voltage"
- note added: "VOUT= 1.235 * (1+R_up/R_down) R_up/R_down needs CAREFUL CALIBRATION such that the VOUT - Schotktky's Vf = 3.300V It can't go below 3.300V. It can be above, but it's less nice if I hotplug USB. R_up R_down Vout 3V3_ext_rail 47k 22k 3.873 V 3.3234 V 100k 47l 3.862 V 3.3126 V"
- note removed: "Main 3V3 LDO, provides up to 500mA (enough for WiFi) Be careful with ADC tempo noise! Set to output strictly more than 3.3V (3.653V) The schotky drops 3.635V to 3.50V which wins over the 3.3V of the USB. When externally powered + USB powered, this means the USB power loses and the ext takes over. ~300 µVrms in adjustable voltage"
- note removed: "VOUT= 1.235 * (1+R_up/R_down)"

Commit message: Lay down PCB with no GND plane breaks
Parts:
- added C21: 100n, easyeda2kicad:C0402, symbol easyeda2kicad:CL05B104KB54PNC
- added F1: MF-R250, easyeda2kicad:FUSE-TH_L12.8-W3.0-P5.80-D1.2-S2.20, symbol easyeda2kicad:MF-R250
- added JP2: SolderJumper_2_Open, Jumper:SolderJumper-2_P1.3mm_Open_TrianglePad1.0x1.5mm, symbol Jumper:SolderJumper_2_Open
- renumbered C21 to C13, R4 to R32, R34 to R33, R3 to R34
Connections:
- net +3.3V: no longer D2.2 (+)
- net S3_3.3V: now also D2.2 (+)
- net VIN_5V: now also C21.2, F1.1, JP2.1 (A); no longer J13.1 (Pin_1)
- net at Q1.1 (G), R31.2: now also C21.1
- new net: F1.2, J13.1 (Pin_1), JP2.2 (B)
Other:
- note added: "The 100nF cap G<->S allows a soft start which limits inrush to the 1000uF bulk cap"
- note added: "The fuse is not going to be added initially, but to not refab I provision in."
- moved on the sheet: J13

Commit message: Finally fabbed v2
Parts:
- removed C_LDO_out1: 2.2uF (225) ±20% 50V, easyeda2kicad:C0805, symbol easyeda2kicad:0805F225M500NT
- removed R33: 1Ω ±1%, easyeda2kicad:R0402, symbol easyeda2kicad:RC0402FR-071RL
- added C_LDO_out1: 2.2uF ±10% 50V, easyeda2kicad:C0805, symbol easyeda2kicad:CL21A225KBQNNNE
- added R33: 1Ω ±1%, easyeda2kicad:R0402, symbol easyeda2kicad:0402WGF100KTCE
- C14, J13, J14, J15, J16, J17, J18, JP1, TP2, TP3: now left out of the parts list
- F1: now not fitted; now left out of the parts list
- renumbered D_S1 to D3, D_PERI1 to D4
Connections:
- net GND: now also R33.1
- net LDO_OUT: now also C_LDO_out1.2
- new net: C_LDO_out1.1, R33.2
