File: boards/one_button/OneButton.kicad_sch (KiCad schematic)
At the start: 18 parts, among them J1 INPUT, J2 OUTPUT, SW1 TS-1187A-B-A-B, U1 CH32V003F4U6

Commit message: Update step models
Parts:
- J1, J2: footprint easyeda2kicad:CONN-TH_B3B-PH-K-S -> easyeda2kicad:CONN-TH_3P-P2.00_S3B-PH-K-S-LF-SN
Changed lines of the file:
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@@
 			)
 		)
-		(property "Footprint" "easyeda2kicad:CONN-TH_B3B-PH-K-S"
+		(property "Footprint" "easyeda2kicad:CONN-TH_3P-P2.00_S3B-PH-K-S-LF-SN"
 			(at 233.68 124.46 0)
 			(hide yes)
@@
 			)
 		)
-		(property "Footprint" "easyeda2kicad:CONN-TH_B3B-PH-K-S"
+		(property "Footprint" "easyeda2kicad:CONN-TH_3P-P2.00_S3B-PH-K-S-LF-SN"
 			(at 243.84 104.14 0)
 			(hide yes)
